File: board/v1/New2.sch (EAGLE design)
At the start: 28 parts, among them IC2 LTC3525, IC3 MCP1703CB, U3 ATMEGA32U4, X1 USB-MICROB, Y1 8MHz

Commit message: example
Parts:
- removed D1: Green, SparkFun:LED0603
- removed SJ1: (no value), jumper:SJ
- added D3: Green, SparkFun:LED0603
- Y1: value 8MHz -> 16MHz
Connections:
- net RXLED renamed D17
- removed net N$8: U3.PD5
- removed net N$9: SJ1.1, U$2.P$6
- new net TXLED: R6.1, U3.PD5
- net A0: now also PORT1.AIO
- net D13: no longer PORT1.DIO
- net D4: now also PORT1.DIO
- net D8: no longer PORT1.AIO
- net GND: no longer D1.C
- net MISO: now also U$1.SDI, U$2.P$5; no longer U$1.SDO, U$2.P$1
- net MOSI: now also U$1.SDO, U$2.P$1; no longer U$1.SDI, U$2.P$5
- net N$6: now also D3.C; no longer D1.A
- net TXO: no longer R6.1
- net VCC: now also D3.A, U$2.P$6; no longer SJ1.2
Other:
- moved on the sheet: R6
