File: board/v1/New_rev1.brd (EAGLE design)
At the start: 21.8 x 22.6 mm, 28 parts, among them IC2 LTC3525, IC3 MCP1703CB, U3 ATMEGA32U4, X1 USB-MICROB, Y1 8MHz

Commit message: example
Parts:
- added D2: (no value), adafruit:SOD-323F
- added Q1: P-MOSFET, SparkFun:SOT23
- C2: value 100n -> 100nF
- C5: value 1u -> 1uF
- C7: value 0.1uF -> 100nF
- R2: value (none) -> 100K
- moved SJ1 0.90 mm to (9.73, 2.30)
- renumbered U$1 to RFM12B
Connections:
- new net N$10: Q1.3, RFM12B.VDD
- net A5: now also D2.A, Q1.1
- net RESET: now also D2.C
- net VCC: now also Q1.2; no longer RFM12B.VDD
Routing:
- net RESET: track 22.1 -> 40.3 mm
- net A5: track 0.00 -> 10.2 mm, vias 0 -> 2
- net N$10: track 0.00 -> 7.18 mm
- net N$9: track 2.12 -> 3.71 mm
- net VCC: track 79.7 -> 78.4 mm
- net VBUS: track 33.3 -> 33.8 mm
- net GND: vias 24 -> 23
