File: board/v1/New_rev1.sch (EAGLE design)
At the start: 28 parts, among them IC2 LTC3525, IC3 MCP1703CB, U3 ATMEGA32U4, X1 USB-MICROB, Y1 8MHz

Commit message: example
Parts:
- added D2: (no value), adafruit:DIODESOD-323F
- added Q1: P-MOSFET, SparkFun:MOSFET-PCHANNEL
- C2: value 100n -> 100nF
- C5: value 1u -> 1uF
- C7: value 0.1uF -> 100nF
- R2: value (none) -> 100K
- renumbered U$1 to RFM12B
Connections:
- new net N$10: Q1.D, RFM12B.VCC
- net A5: now also D2.A, Q1.G
- net RESET: now also D2.C
- net VCC: now also Q1.S; no longer RFM12B.VCC
Other:
- moved on the sheet: C2
