File: board/v1/New.brd (EAGLE design)
At the start: 21.8 x 22.6 mm, 28 parts, among them IC2 LTC3525, IC3 MCP1703CB, U3 ATMEGA32U4, X1 USB-MICROB, Y1 8MHz

Commit message: Revert "example"
This reverts commit 1f9ad8d22b45befcb35b8a9bb4ed2c9c1b9cff3c.
Parts:
- Y1: value 8MHz -> 16MHz
Changed lines of the file:
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@@
 <element name="R6" library="SparkFun" package="0402-RES" value="330" x="12.541" y="6.391" rot="R180"/>
 <element name="U3" library="SparkFun" package="QFN-44-NOPAD" value="ATMEGA32U4" x="13.081" y="12.7" rot="R315"/>
-<element name="Y1" library="SparkFun" package="CRYSTAL-SMD-5X3" value="8MHz" x="3.937" y="9.525" rot="R270"/>
+<element name="Y1" library="SparkFun" package="CRYSTAL-SMD-5X3" value="16MHz" x="3.937" y="9.525" rot="R270"/>
 <element name="C8" library="SparkFun" package="0402-CAP" value="22pF" x="4.445" y="5.842" rot="R180"/>
 <element name="C9" library="SparkFun" package="0402-CAP" value="22pF" x="3.302" y="13.081"/>
