File: board/v3/Funky_v3_r3.brd (EAGLE design)
At the start: 21.8 x 22.6 mm, 43 parts, among them IC2 LTC3525, IC3 MCP1703CB, Q1 P-MOSFET, U3 ATMEGA32U4, Y1 8MHz

Commit message: Update the project folder to latet
Parts:
- renumbered IC3 to TOREX-XC6206
Changed lines of the file:
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@@
 <?xml version="1.0" encoding="utf-8"?>
 <!DOCTYPE eagle SYSTEM "eagle.dtd">
-<eagle version="6.3">
+<eagle version="6.1">
 <drawing>
 <settings>
@@
 <text x="12.462" y="20.134" size="1.016" layer="21">+3V3</text>
 <text x="16.505" y="21.402" size="1.016" layer="21">Ant.</text>
-<text x="18.688" y="16.896" size="0.8128" layer="21" font="vector">5V</text>
-<text x="17.728" y="14.4" size="0.8128" layer="21" font="vector">D11</text>
+<text x="18.432" y="14.208" size="0.8128" layer="21" font="vector">5V</text>
+<text x="17.792" y="17.088" size="0.8128" layer="21" font="vector">D11</text>
 <text x="17.6" y="11.84" size="0.8128" layer="21" font="vector">GND</text>
 <text x="17.6" y="8.704" size="0.8128" layer="21" font="vector">VCC</text>
@@
 </class>
 </classes>
-<designrules name="default">
+<designrules>
 <description language="de">&lt;b&gt;EAGLE Design Rules Prototypen  für PCB-POOL(R)&lt;/b&gt;
 &lt;p&gt;
@@
 <element name="IC2" library="JeeLabs" package="SC70" value="LTC3525" x="16.579" y="4.384" rot="R180"/>
 <element name="L1" library="SparkFun" package="1210" value="10 µH" x="15.614" y="2.095" rot="MR180"/>
-<element name="IC3" library="linear" package="SOT23" value="MCP1703CB" x="3.048" y="21.463" rot="MR90"/>
+<element name="TOREX-XC6206" library="linear" package="SOT23" value="MCP1703CB" x="3.048" y="21.463" rot="MR90"/>
 <element name="C5" library="rcl" package="C0603K" value="1uF" x="11.56" y="20.016"/>
 <element name="C6" library="rcl" package="C0603K" value="1u" x="9.525" y="21.463" rot="MR270"/>
@@
 <contactref element="C6" pad="1"/>
 <contactref element="PAD10" pad="1"/>
-<contactref element="IC3" pad="2"/>
+<contactref element="TOREX-XC6206" pad="2"/>
 <wire x1="12.3169" y1="12.1841" x2="12.476" y2="12.025" width="0.254" layer="16"/>
 <wire x1="12.476" y1="12.025" x2="16.6437" y2="12.025" width="0.254" layer="16"/>
@@
 <contactref element="C6" pad="2"/>
 <contactref element="C5" pad="2"/>
-<contactref element="IC3" pad="1"/>
+<contactref element="TOREX-XC6206" pad="1"/>
 <contactref element="C7" pad="1"/>
 <contactref element="C8" pad="2"/>
@@
 </signal>
 <signal name="VBUS" class="1">
-<contactref element="IC3" pad="3"/>
+<contactref element="TOREX-XC6206" pad="3"/>
 <contactref element="C5" pad="1"/>
 <contactref element="U3" pad="7"/>
